File: wbz451pe.brd (EAGLE design)
At the start: 160 x 45.4 mm, 1 part, among them U1 WBZ451PE-IWBZ451_MCH

Commit message: up
Parts:
- moved U1 1.27 mm to (26.7, 39.4)
Connections:
- new net GND: U1.1, U1.11, U1.19, U1.2, U1.26, U1.40, U1.41, U1.42, U1.43, U1.44, U1.45, U1.46, U1.47, U1.48, U1.8
Routing:
- added copper zone on layer 1, net GND
- added copper zone on layer 16, net GND
- added copper zone on layer 2, net GND
Changed lines of the file:
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@@
 <layers>
 <layer number="1" name="Top" color="4" fill="1" visible="yes" active="yes"/>
-<layer number="2" name="Route2" color="16" fill="1" visible="no" active="no"/>
+<layer number="2" name="Route2" color="16" fill="1" visible="yes" active="yes"/>
 <layer number="3" name="Route3" color="17" fill="1" visible="no" active="no"/>
 <layer number="4" name="Route4" color="18" fill="1" visible="no" active="no"/>
@@
 <layer number="13" name="Route13" color="21" fill="1" visible="no" active="no"/>
 <layer number="14" name="Route14" color="22" fill="1" visible="no" active="no"/>
-<layer number="15" name="Route15" color="23" fill="1" visible="no" active="no"/>
+<layer number="15" name="Route15" color="23" fill="1" visible="yes" active="yes"/>
 <layer number="16" name="Bottom" color="1" fill="1" visible="yes" active="yes"/>
 <layer number="17" name="Pads" color="2" fill="1" visible="yes" active="yes"/>
@@
 </class>
 </classes>
-<designrules name="default">
+<designrules name="default *">
 <description language="de">&lt;b&gt;EAGLE Design Rules&lt;/b&gt;
 &lt;p&gt;
@@
 necessary adjustments and save your customized
 design rules under a new name.</description>
-<param name="layerSetup" value="(1*16)"/>
+<param name="layerSetup" value="(1+2*15+16)"/>
 <param name="mtCopper" value="0.035mm 0.035mm 0.035mm 0.035mm 0.035mm 0.035mm 0.035mm 0.035mm 0.035mm 0.035mm 0.035mm 0.035mm 0.035mm 0.035mm 0.035mm 0.035mm"/>
 <param name="mtIsolate" value="1.5mm 0.15mm 0.2mm 0.15mm 0.2mm 0.15mm 0.2mm 0.15mm 0.2mm 0.15mm 0.2mm 0.15mm 0.2mm 0.15mm 0.2mm"/>
@@
 <param name="tpViaShape" value="round"/>
 <param name="PrefDir.1" value="a"/>
-<param name="PrefDir.2" value="0"/>
+<param name="PrefDir.2" value="a"/>
 <param name="PrefDir.3" value="0"/>
 <param name="PrefDir.4" value="0"/>
@@
 <param name="PrefDir.13" value="0"/>
 <param name="PrefDir.14" value="0"/>
-<param name="PrefDir.15" value="0"/>
+<param name="PrefDir.15" value="a"/>
 <param name="PrefDir.16" value="a"/>
 <param name="cfVia" value="8"/>
@@
 </autorouter>
 <elements>
-<element name="U1" library="2024-05-29_22-27-45_Library" package="WBZ451_MCH" value="WBZ451PE-IWBZ451_MCH" x="27.94" y="39.37" smashed="yes">
-<attribute name="COPYRIGHT" value="Copyright (C) 2024 Ultra Librarian. All rights reserved." x="62.23" y="24.13" size="1.778" layer="27" display="off"/>
-<attribute name="MANUFACTURER_PART_NUMBER" value="WBZ451PE-I" x="62.23" y="24.13" size="1.778" layer="27" display="off"/>
-<attribute name="MFR_NAME" value="Microchip" x="62.23" y="24.13" size="1.778" layer="27" display="off"/>
-<attribute name="NAME" x="27.2088" y="42.545" size="1.27" layer="27" ratio="6"/>
-<attribute name="VALUE" x="18.5912" y="51.435" size="1.27" layer="27" ratio="6"/>
+<element name="U1" library="2024-05-29_22-27-45_Library" package="WBZ451_MCH" value="WBZ451PE-IWBZ451_MCH" x="26.67" y="39.37" smashed="yes">
+<attribute name="COPYRIGHT" value="Copyright (C) 2024 Ultra Librarian. All rights reserved." x="26.67" y="39.37" size="1.778" layer="27" display="off"/>
+<attribute name="MANUFACTURER_PART_NUMBER" value="WBZ451PE-I" x="26.67" y="39.37" size="1.778" layer="27" display="off"/>
+<attribute name="MFR_NAME" value="Microchip" x="26.67" y="39.37" size="1.778" layer="27" display="off"/>
+<attribute name="NAME" x="23.3988" y="38.735" size="1.27" layer="27" ratio="6"/>
+<attribute name="VALUE" x="24.9412" y="38.735" size="1.27" layer="27" ratio="6"/>
 </element>
 </elements>
 <signals>
+<signal name="GND">
+<polygon width="0.1524" layer="1">
+<vertex x="11.43" y="43.18"/>
+<vertex x="43.18" y="43.18"/>
+<vertex x="43.18" y="22.86"/>
+<vertex x="12.7" y="22.86"/>
+<vertex x="11.43" y="22.86"/>
+</polygon>
+<polygon width="0.1524" layer="2">
+<vertex x="1.27" y="43.18"/>
+<vertex x="157.48" y="43.18"/>
+<vertex x="157.48" y="1.27"/>
+<vertex x="1.27" y="1.27"/>
+</polygon>
+<polygon width="0.1524" layer="16">
+<vertex x="1.27" y="43.18"/>
+<vertex x="157.48" y="43.18"/>
+<vertex x="157.48" y="1.27"/>
+<vertex x="1.27" y="1.27"/>
+</polygon>
+<contactref element="U1" pad="1"/>
+<contactref element="U1" pad="2"/>
+<contactref element="U1" pad="8"/>
+<contactref element="U1" pad="11"/>
+<contactref element="U1" pad="19"/>
+<contactref element="U1" pad="26"/>
+<contactref element="U1" pad="43"/>
+<contactref element="U1" pad="40"/>
+<contactref element="U1" pad="41"/>
+<contactref element="U1" pad="46"/>
+<contactref element="U1" pad="47"/>
+<contactref element="U1" pad="44"/>
+<contactref element="U1" pad="42"/>
+<contactref element="U1" pad="48"/>
+<contactref element="U1" pad="45"/>
+</signal>
 <signal name="VDD_A">
 <contactref element="U1" pad="7"/>

Commit message: up
Parts:
- added C1, C5, C6: 0.1uf, rcl:C0805
- added C2, C3, C4, C7: 10uf, rcl:C0805
- added PICKIT: PICKIT, pinhead:1X08
- added R1, R3, R4, R5, R6: 0, rcl:M0805
- added R2: 10k, rcl:M0805
Connections:
- removed net VDD_2: U1.27
- removed net VDD_A: U1.7
- new net CM4_SWCLK: PICKIT.5, R4.1
- new net CM4_SWDIO: PICKIT.8, R5.1, R6.2
- new net CM4_SWO: PICKIT.4, R3.1
- new net MCLR_L: C1.1, PICKIT.6, R1.1, R2.1
- new net N$1: R1.2, U1.3
- new net SWCLK: R4.2, U1.14
- new net SWDIO: R5.2, U1.15
- new net SWO: R3.2, U1.13
- net GND: now also C1.2, C2.2, C3.2, C4.2, C5.2, C6.2, C7.2, PICKIT.3
- net VDD: now also C2.1, C3.1, C4.1, C5.1, C6.1, C7.1, PICKIT.2, R2.2, R6.1, U1.27, U1.7
Routing:
- net VDD: track 0.00 -> 114.1 mm
- net MCLR_L: track 0.00 -> 49.3 mm
- net CM4_SWDIO: track 0.00 -> 25.9 mm
- net GND: track 0.00 -> 19.1 mm, vias 0 -> 4
- net CM4_SWCLK: track 0.00 -> 18.4 mm
- net CM4_SWO: track 0.00 -> 14.7 mm
- net N$1: track 0.00 -> 8.77 mm, vias 0 -> 2
- net SWO: track 0.00 -> 8.42 mm
- net SWCLK: track 0.00 -> 6.27 mm
- net SWDIO: track 0.00 -> 5.57 mm
Other:
- board size 160 x 45.4 mm -> 104.1 x 45.4 mm

Commit message: up
Parts:
- added C8: 0.1uf, rcl:C0805
- added IC1: SST26VF064B-104I_MF, SST26VF064B-104I_MF:SON127P600X500X80-9N
- added R10, R11, R9: 0, rcl:M0805
- added R12: 0, rcl:R0603
- added R13, R14, R15, R16, R17: 33, rcl:R0603
- added R18, R19, R20: 100k, rcl:R0603
- added R7: 10k, rcl:M0805
- added R8: 680, rcl:M0805
- added S1: B3W-9000-Y1N, SamacSys_Parts:B3W-9_1-LED
- added SWD_DEBUG: EHF-105-01-L-D-SM-LC, EHF-105-01-L-D-SM-LC:EHF-105-01-XX-D-SM-LC
- added TP1, TP2, TP3: TPPAD1-13, testpad:P1-13
- R6: value 0 -> 10k
Connections:
- new net BLED: R11.1, TP3.TP
- new net GLED: R10.1, TP2.TP
- new net N$10: IC1.6, R16.1
- new net N$11: IC1.5, R17.1, R20.1
- new net N$2: R9.2, U1.4
- new net N$3: R8.1, S1.5
- new net N$4: R10.2, U1.5
- new net N$5: R11.2, U1.6
- new net N$6: IC1.1, R12.2, R18.2
- new net N$7: IC1.2, R13.2
- new net N$8: IC1.3, R14.2
- new net N$9: IC1.7, R15.1, R19.1
- new net QCS: R12.1, U1.17
- new net QSCK: R16.2, U1.18
- new net QSPI0: R17.2, U1.22
- new net QSPI1: R13.1, U1.23
- new net QSPI2: R14.1, U1.20
- new net QSPI3: R15.2, U1.21
- new net RLED: R9.1, TP1.TP
- net CM4_SWCLK: now also R7.1, SWD_DEBUG.4
- net CM4_SWDIO: now also SWD_DEBUG.2
- net CM4_SWO: now also SWD_DEBUG.6
- net GND: now also C8.2, IC1.4, IC1.9, S1.3, S1.4, S1.6, SWD_DEBUG.3, SWD_DEBUG.5, SWD_DEBUG.9
- net MCLR_L: now also S1.1, S1.2, SWD_DEBUG.10
- net SWO: now also R8.2
- net VDD: now also C8.1, IC1.8, R18.1, R19.2, R20.2, R7.2, SWD_DEBUG.1
Routing:
- net VDD: track 114.1 -> 190.6 mm
- net MCLR_L: track 49.3 -> 108.2 mm
- net N$5: track 0.00 -> 35.6 mm, vias 0 -> 2
- net N$9: track 0.00 -> 35.3 mm, vias 0 -> 2
- net CM4_SWCLK: track 18.4 -> 53.2 mm, vias 0 -> 1
- net N$11: track 0.00 -> 33.3 mm
- net N$3: track 0.00 -> 33.1 mm, vias 0 -> 1
- net QSPI0: track 0.00 -> 29.0 mm
- net N$10: track 0.00 -> 27.1 mm
- net N$8: track 0.00 -> 24.1 mm
- net N$6: track 0.00 -> 20.1 mm, vias 0 -> 3
- net SWO: track 8.42 -> 28.4 mm, vias 0 -> 2
- net CM4_SWDIO: track 25.9 -> 44.5 mm, vias 0 -> 1
- net QSPI3: track 0.00 -> 17.5 mm, vias 0 -> 2
- net CM4_SWO: track 14.7 -> 31.0 mm
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