File: wbz451pe.sch (EAGLE design)
At the start: 1 part, among them U1 WBZ451PE-IWBZ451_MCH

Commit message: up
Connections:
- new net GND: U1.EGND, U1.GND, U1.GND_2, U1.GND_3, U1.GND_4, U1.GND_5, U1.GND_6
Other:
- moved on the sheet: U1
Changed lines of the file:
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@@
 </busses>
 <nets>
+<net name="GND" class="0">
+<segment>
+<wire x1="60.96" y1="66.04" x2="55.88" y2="66.04" width="0.1524" layer="91"/>
+<label x="55.88" y="66.04" size="1.778" layer="95"/>
+<pinref part="U1" gate="A" pin="GND_2"/>
+<junction x="60.96" y="66.04"/>
+</segment>
+<segment>
+<wire x1="60.96" y1="63.5" x2="55.88" y2="63.5" width="0.1524" layer="91"/>
+<label x="55.88" y="63.5" size="1.778" layer="95"/>
+<pinref part="U1" gate="A" pin="GND_3"/>
+<junction x="60.96" y="63.5"/>
+</segment>
+<segment>
+<wire x1="60.96" y1="48.26" x2="55.88" y2="48.26" width="0.1524" layer="91"/>
+<label x="55.88" y="48.26" size="1.778" layer="95"/>
+<pinref part="U1" gate="A" pin="GND_4"/>
+<junction x="60.96" y="48.26"/>
+</segment>
+<segment>
+<wire x1="60.96" y1="40.64" x2="55.88" y2="40.64" width="0.1524" layer="91"/>
+<label x="55.88" y="40.64" size="1.778" layer="95"/>
+<pinref part="U1" gate="A" pin="GND_5"/>
+<junction x="60.96" y="40.64"/>
+</segment>
+<segment>
+<wire x1="60.96" y1="20.32" x2="55.88" y2="20.32" width="0.1524" layer="91"/>
+<label x="55.88" y="20.32" size="1.778" layer="95"/>
+<pinref part="U1" gate="A" pin="GND_6"/>
+<junction x="60.96" y="20.32"/>
+</segment>
+<segment>
+<wire x1="96.52" y1="30.48" x2="104.14" y2="30.48" width="0.1524" layer="91"/>
+<label x="101.6" y="30.48" size="1.778" layer="95"/>
+<pinref part="U1" gate="A" pin="GND"/>
+<junction x="96.52" y="30.48"/>
+</segment>
+<segment>
+<wire x1="96.52" y1="66.04" x2="106.68" y2="66.04" width="0.1524" layer="91"/>
+<label x="101.6" y="66.04" size="1.778" layer="95"/>
+<pinref part="U1" gate="A" pin="EGND"/>
+<junction x="96.52" y="66.04"/>
+</segment>
+</net>
 </nets>
 </sheet>

Commit message: up
Parts:
- added C1, C5, C6: 0.1uf, rcl:C-USC0805
- added C2, C3, C4, C7: 10uf, rcl:C-USC0805
- added PICKIT: PICKIT, pinhead:PINHD-1X8
- added R1, R3, R4, R5, R6: 0, rcl:R-US_M0805
- added R2: 10k, rcl:R-US_M0805
Connections:
- new net CM4_SWCLK: PICKIT.5, R4.1
- new net CM4_SWDIO: PICKIT.8, R5.1, R6.2
- new net CM4_SWO: PICKIT.4, R3.1
- new net MCLR_L: C1.1, PICKIT.6, R1.1, R2.1
- new net N$1: R1.2, U1.NMCLR
- new net SWCLK: R4.2, U1.PB8
- new net SWDIO: R5.2, U1.PB9
- new net SWO: R3.2, U1.PB7
- new net VDD: C2.1, C3.1, C4.1, C5.1, C6.1, C7.1, PICKIT.2, R2.2, R6.1, U1.VDD, U1.VDD_2, U1.VDD_A
- net GND: now also C1.2, C2.2, C3.2, C4.2, C5.2, C6.2, C7.2, PICKIT.3

Commit message: up
Parts:
- added C8: 0.1uf, rcl:C-USC0805
- added IC1: SST26VF064B-104I_MF, SST26VF064B-104I_MF:SST26VF064B-104I_MF
- added R10, R11, R9: 0, rcl:R-US_M0805
- added R12: 0, rcl:R-US_R0603
- added R13, R14, R15, R16, R17: 33, rcl:R-US_R0603
- added R18, R19, R20: 100k, rcl:R-US_R0603
- added R7: 10k, rcl:R-US_M0805
- added R8: 680, rcl:R-US_M0805
- added S1: B3W-9000-Y1N, SamacSys_Parts:B3W-9000-Y1N
- added SWD_DEBUG: EHF-105-01-L-D-SM-LC, EHF-105-01-L-D-SM-LC:EHF-105-01-L-D-SM-LC
- added TP1, TP2, TP3: TPPAD1-13, testpad:TPPAD1-13
- R6: value 0 -> 10k
Connections:
- new net BLED: R11.1, TP3.TP
- new net GLED: R10.1, TP2.TP
- new net N$10: IC1.SCK, R16.1
- new net N$11: IC1.SI/SIO0, R17.1, R20.1
- new net N$2: R9.2, U1.PB0
- new net N$3: R8.1, S1.+
- new net N$4: R10.2, U1.PB3
- new net N$5: R11.2, U1.PB5
- new net N$6: IC1.CE#, R12.2, R18.2
- new net N$7: IC1.SO/SIO1, R13.2
- new net N$8: IC1.WP#/SIO2, R14.2
- new net N$9: IC1.HOLD/SIO3, R15.1, R19.1
- new net QCS: R12.1, U1.PB10
- new net QSCK: R16.2, U1.PB11
- new net QSPI0: R17.2, U1.PB12
- new net QSPI1: R13.1, U1.PB13
- new net QSPI2: R14.1, U1.PA0
- new net QSPI3: R15.2, U1.PA1
- new net RLED: R9.1, TP1.TP
- net CM4_SWCLK: now also R7.1, SWD_DEBUG.4
- net CM4_SWDIO: now also SWD_DEBUG.2
- net CM4_SWO: now also SWD_DEBUG.6
- net GND: now also C8.2, IC1.EP, IC1.VSS, S1.-, S1.3, S1.4, SWD_DEBUG.3, SWD_DEBUG.5, SWD_DEBUG.9
- net MCLR_L: now also S1.1, S1.2, SWD_DEBUG.10
- net SWO: now also R8.2
- net VDD: now also C8.1, IC1.VDD, R18.1, R19.2, R20.2, R7.2, SWD_DEBUG.1
